File: hardware/KiCad/clippi/clippi.kicad_sch (KiCad schematic)
At the start: 19 parts, among them J1 GPIO, J2 Conn_01x16_Pin, Q1 BSS138

Commit message: fix pi hat board/schematic to ensure 3.3v is supplied to the logic shifter, that got missed
Parts:
- renumbered 0v to 0v2, 5v to 5v1, SCL to SCL1, SDA to SDA1
Connections:
- net +3.3V is gone; now on net +3V3: Q1.1 (G), R3.2
Changed lines of the file:
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@@
   (junction (at 67.31 166.37) (diameter 0) (color 0 0 0 0)
   )
+  (junction (at 40.64 45.72) (diameter 0) (color 0 0 0 0)
+  )
   (junction (at 46.99 166.37) (diameter 0) (color 0 0 0 0)
   )
@@
     (stroke (width 0) (type solid))
   )
-  (wire (pts (xy 46.99 139.7) (xy 46.99 147.32))
-    (stroke (width 0) (type default))
-  )
   (wire (pts (xy 38.1 166.37) (xy 46.99 166.37))
     (stroke (width 0) (type default))
@@
     (stroke (width 0) (type solid))
   )
+  (wire (pts (xy 40.64 45.72) (xy 45.72 45.72))
+    (stroke (width 0) (type default))
+  )
   (wire (pts (xy 58.42 43.18) (xy 85.09 43.18))
     (stroke (width 0) (type solid))
@@
     (stroke (width 0) (type default))
   )
-  (wire (pts (xy 40.64 45.72) (xy 45.72 45.72))
+  (wire (pts (xy 40.64 45.72) (xy 39.37 45.72))
     (stroke (width 0) (type solid))
   )
@@
     (stroke (width 0) (type solid))
   )
+  (wire (pts (xy 46.99 142.24) (xy 46.99 147.32))
+    (stroke (width 0) (type default))
+  )
   (wire (pts (xy 193.04 87.63) (xy 199.39 87.63))
     (stroke (width 0) (type default))
@@
     (effects (font (size 1.27 1.27)) (justify right bottom))
   )
+  (label "3.3v jumper" (at 45.72 25.4 180) (fields_autoplaced)
+    (effects (font (size 1.27 1.27)) (justify right bottom))
+  )
   (label "GPIO22" (at 16.51 43.18 0) (fields_autoplaced)
     (effects (font (size 1.27 1.27)) (justify left bottom))
@@
   (label "GPIO18{slash}PCM.CLK" (at 38.1 166.37 180) (fields_autoplaced)
     (effects (font (size 1.27 1.27)) (justify right bottom))
+  )
+  (label "3.3v jumper" (at 46.99 142.24 90) (fields_autoplaced)
+    (effects (font (size 1.27 1.27)) (justify left bottom))
   )
   (label "GPIO11{slash}SPI0.SCLK" (at 16.51 53.34 0) (fields_autoplaced)
@@
   (symbol (lib_id "Connector:Conn_01x01_Pin") (at 191.77 30.48 0) (unit 1)
     (in_bom yes) (on_board yes) (dnp no)
-    (property "Reference" "SDA" (at 192.405 25.4 0)
+    (property "Reference" "SDA1" (at 192.405 25.4 0)
       (effects (font (size 1.27 1.27)) hide)
     )
@@
       (project "clippi"
         (path "/e63e39d7-6ac0-4ffd-8aa3-1841a4541b55"
-          (reference "SDA") (unit 1)
+          (reference "SDA1") (unit 1)
         )
       )
@@
     )
   )
-  (symbol (lib_name "+3.3V_1") (lib_id "power:+3.3V") (at 46.99 139.7 0) (unit 1)
-    (in_bom yes) (on_board yes) (dnp no) (fields_autoplaced)
-    (property "Reference" "#PWR015" (at 46.99 143.51 0)
-      (effects (font (size 1.27 1.27)) hide)
-    )
-    (property "Value" "+3.3V" (at 46.99 134.62 0)
-      (effects (font (size 1.27 1.27)))
-    )
-    (property "Footprint" "" (at 46.99 139.7 0)
-      (effects (font (size 1.27 1.27)) hide)
-    )
-    (property "Datasheet" "" (at 46.99 139.7 0)
-      (effects (font (size 1.27 1.27)) hide)
-    )
-    (pin "1")
-    (instances
-      (project "clippi"
-        (path "/e63e39d7-6ac0-4ffd-8aa3-1841a4541b55"
-          (reference "#PWR015") (unit 1)
-        )
-      )
-    )
-  )
   (symbol (lib_id "Connector:Conn_01x01_Pin") (at 113.03 143.51 0) (unit 1)
     (in_bom yes) (on_board yes) (dnp no)
@@
   (symbol (lib_id "Connector:Conn_01x01_Pin") (at 191.77 33.02 0) (unit 1)
     (in_bom yes) (on_board yes) (dnp no)
-    (property "Reference" "SCL" (at 192.405 27.94 0)
+    (property "Reference" "SCL1" (at 192.405 27.94 0)
       (effects (font (size 1.27 1.27)) hide)
     )
@@
       (project "clippi"
         (path "/e63e39d7-6ac0-4ffd-8aa3-1841a4541b55"
-          (reference "SCL") (unit 1)
+          (reference "SCL1") (unit 1)
         )
       )
@@
   (symbol (lib_id "Connector:Conn_01x01_Pin") (at 191.77 25.4 0) (unit 1)
     (in_bom yes) (on_board yes) (dnp no)
-    (property "Reference" "5v" (at 192.405 20.32 0)
+    (property "Reference" "5v1" (at 192.405 20.32 0)
       (effects (font (size 1.27 1.27)) hide)
     )
@@
       (project "clippi"
         (path "/e63e39d7-6ac0-4ffd-8aa3-1841a4541b55"
-          (reference "5v") (unit 1)
+          (reference "5v1") (unit 1)
         )
       )
@@
   (symbol (lib_id "Connector:Conn_01x01_Pin") (at 191.77 27.94 0) (unit 1)
     (in_bom yes) (on_board yes) (dnp no)
-    (property "Reference" "0v" (at 192.405 22.86 0)
+    (property "Reference" "0v2" (at 192.405 22.86 0)
       (effects (font (size 1.27 1.27)) hide)
     )
@@
       (project "clippi"
         (path "/e63e39d7-6ac0-4ffd-8aa3-1841a4541b55"
-          (reference "0v") (unit 1)
-        )
-      )
+          (reference "0v2") (unit 1)
+        )
+      )
